Commit message: Updated

File: ROS2_sim/install/simple_robot/share/simple_robot/urdf/simple_robot.urdf (robot description, URDF)
Before this commit: robot simple_robot, 3 links, 2 joints
Links:
- added link link2_2; visual box size=0.2 0.025 0.025
- link link2_1: geometry visual cylinder length=0.1 radius=0.025
- link plato_giro: geometry visual cylinder length=0.05 radius=0.025
Joints:
- added joint EL2: type fixed, parent link2_1, child link2_2, origin xyz=0.2 0 0 rpy=0 0 0, axis 0 0 1
- joint J1: origin xyz=0 0 0.075 -> xyz=0 0 0.1
- joint J2: origin xyz=0 0 0.035 rpy=1.570796 0 0 -> xyz=0 0 0 rpy=1.570796 0 0

Commit message: Updated

File: ROS2_sim/install/simple_robot/share/simple_robot/urdf/simple_robot.urdf (robot description, URDF)
Before this commit: robot simple_robot, 4 links, 3 joints
Links:
- removed link plato_giro
- added link link1_2; visual cylinder length=0.5 radius=0.25
- link base_link: geometry visual box size=1 1 0.5
- link link2_1: geometry visual cylinder length=1 radius=0.25
- link link2_2: geometry visual box size=2 0.25 0.25
Joints:
- joint EL2: origin xyz=0.2 0 0 rpy=0 0 0 -> xyz=2 0 0 rpy=0 0 0
- joint J1: axis 0 0 0.1 -> 0 0 1; child plato_giro -> link1_2; origin xyz=0 0 0.1 -> xyz=0 0 0.75
- joint J2: origin xyz=0 0 0 rpy=1.570796 0 0 -> xyz=0 0 0.5 rpy=1.570796 0 0; parent plato_giro -> link1_2

Commit message: Updated

File: ROS2_sim/install/simple_robot/share/simple_robot/urdf/simple_robot.urdf (robot description, URDF)
Before this commit: robot simple_robot, 4 links, 3 joints
Links:
- added link link3_1; visual cylinder length=0.5 radius=0.25
- added link link3_2; visual box size=2 0.25 0.25
- link link2_1: geometry visual cylinder length=0.5 radius=0.25
Joints:
- added joint EL3: type fixed, parent link3_1, child link3_2, origin xyz=2 0 0 rpy=0 0 0, axis 0 0 1
- added joint J3: type continuous, parent link2_2, child link3_1, origin xyz=0 0 0 rpy=0 0 0, axis 0 0 1
- joint J1: origin xyz=0 0 0.75 -> xyz=0 0 0.75 rpy=0 0 0
