Commit message: updated SCARA 3DOF

File: ROS2_sim/src/scara_3DOF/urdf/scara_3DOF.urdf (robot description, URDF)
Before this commit: robot simple_robot, 7 links, 6 joints
Joints:
- joint J2: limit (none) -> lower=0.0 upper=1.8 effort=1000.0 velocity=2.0; type continuous -> revolute
- joint J3: limit (none) -> lower=-0.8 upper=0.1 effort=1000.0 velocity=1.0; type continuous -> prismatic
