Commit message: 6_dof ros_controllers

File: ROS2_sim/src/robot_6dof_pkg/urdf/Robot.urdf (robot description, URDF)
Before this commit: robot Robot, 7 links, 6 joints
Links:
- added link world
Joints:
- added joint fixed_base: type fixed, parent world, child Base
- joint Base__to__link_1: limit (none) -> lower=-3.14 upper=3.14 effort=1000.0 velocity=6.0
- joint link_1__to__link_2: limit (none) -> lower=-1.57 upper=0.0 effort=1000.0 velocity=6.0
- joint link_2__to__link_3: limit (none) -> lower=-1.57 upper=0.0 effort=1000.0 velocity=6.0
- joint link_3__to__link_4: limit (none) -> lower=-3.14 upper=3.14 effort=1000.0 velocity=6.0; origin xyz=0.14 0.0 0.005 rpy=-1.5707963267948968 0 1.5707963267948966 -> xyz=0.14 0.0 0.005 rpy=-1.5707963267948968 0 1.5707963267948968
- joint link_4__to__link_5: limit (none) -> lower=0.0 upper=1.57 effort=1000.0 velocity=6.0
- joint link_5__to__link_6: limit (none) -> lower=-3.14 upper=3.14 effort=1000.0 velocity=6.0
